File: pcb.brd (EAGLE design)
At the start: 303.8 x 96.2 mm, 138 parts

Commit message: updated matrix and streched pcb
Connections:
- new net N$84: MACRO_0.MX2, MACRO_1.MX2, MACRO_2.MX2
- net N$76: no longer MACRO_0.MX2
- net N$78: no longer MACRO_1.MX2
- net N$83: no longer MACRO_2.MX2
- net ROW0: now also D68.C
- net ROW1: now also D69.C
- net ROW4: no longer D68.C, D69.C
Other:
- board size 303.8 x 96.2 mm -> 307.8 x 96.2 mm
Changed lines of the file:
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@@
 <board>
 <plain>
-<wire x1="313.80035" y1="102.25" x2="313.80035" y2="12.05" width="0.001" layer="20"/>
-<wire x1="313.80035" y1="102.25" x2="311.80035" y2="104.25" width="0.001" layer="20" curve="90"/>
-<wire x1="311.80035" y1="10.05" x2="12.05" y2="10.05" width="0.001" layer="20"/>
-<wire x1="10.05" y1="12.05" x2="12.05" y2="10.05" width="0.001" layer="20" curve="90"/>
-<wire x1="311.80035" y1="10.05" x2="313.80035" y2="12.05" width="0.001" layer="20" curve="90"/>
-<wire x1="10.05" y1="12.05" x2="10.05" y2="102.25" width="0.001" layer="20"/>
-<wire x1="12.05" y1="104.25" x2="10.05" y2="102.25" width="0.001" layer="20" curve="90"/>
-<wire x1="23.57501875" y1="106.25" x2="23.57501875" y2="104.25" width="0.001" layer="20"/>
-<wire x1="33.57501875" y1="106.25" x2="33.57501875" y2="104.25" width="0.001" layer="20"/>
-<wire x1="23.57501875" y1="106.25" x2="33.57501875" y2="106.25" width="0.001" layer="20"/>
-<wire x1="156.92516875" y1="106.25" x2="156.92516875" y2="104.25" width="0.001" layer="20"/>
-<wire x1="166.92516875" y1="106.25" x2="166.92516875" y2="104.25" width="0.001" layer="20"/>
-<wire x1="156.92516875" y1="106.25" x2="166.92516875" y2="106.25" width="0.001" layer="20"/>
-<wire x1="290.06295" y1="106.25" x2="290.06295" y2="104.25" width="0.001" layer="20"/>
-<wire x1="300.06295" y1="106.25" x2="300.06295" y2="104.25" width="0.001" layer="20"/>
-<wire x1="290.06295" y1="106.25" x2="300.06295" y2="106.25" width="0.001" layer="20"/>
-<wire x1="23.57501875" y1="104.25" x2="12.05" y2="104.25" width="0.001" layer="20"/>
-<wire x1="33.57501875" y1="104.25" x2="156.92516875" y2="104.25" width="0.001" layer="20"/>
-<wire x1="166.92516875" y1="104.25" x2="290.06295" y2="104.25" width="0.001" layer="20"/>
-<wire x1="300.06295" y1="104.25" x2="311.80035" y2="104.25" width="0.001" layer="20"/>
 <wire x1="297.80045" y1="26.04953125" x2="311.79945" y2="26.04953125" width="0.001" layer="49"/>
 <wire x1="311.79945" y1="26.04953125" x2="311.79945" y2="12.05006875" width="0.001" layer="49"/>
@@
 <wire x1="0" y1="0" x2="0" y2="95.25" width="0.001" layer="49"/>
 <wire x1="0" y1="95.25" x2="19.05" y2="95.25" width="0.001" layer="49"/>
+<wire x1="315.80035" y1="102.25" x2="315.80035" y2="12.05" width="0.001" layer="20"/>
+<wire x1="315.80035" y1="102.25" x2="313.80035" y2="104.25" width="0.001" layer="20" curve="90"/>
+<wire x1="313.80035" y1="10.05" x2="10.05" y2="10.05" width="0.001" layer="20"/>
+<wire x1="8.05" y1="12.05" x2="10.05" y2="10.05" width="0.001" layer="20" curve="90"/>
+<wire x1="313.80035" y1="10.05" x2="315.80035" y2="12.05" width="0.001" layer="20" curve="90"/>
+<wire x1="8.05" y1="12.05" x2="8.05" y2="102.25" width="0.001" layer="20"/>
+<wire x1="10.05" y1="104.25" x2="8.05" y2="102.25" width="0.001" layer="20" curve="90"/>
+<wire x1="23.57501875" y1="106.25" x2="23.57501875" y2="104.25" width="0.001" layer="20"/>
+<wire x1="33.57501875" y1="106.25" x2="33.57501875" y2="104.25" width="0.001" layer="20"/>
+<wire x1="23.57501875" y1="106.25" x2="33.57501875" y2="106.25" width="0.001" layer="20"/>
+<wire x1="156.92516875" y1="106.25" x2="156.92516875" y2="104.25" width="0.001" layer="20"/>
+<wire x1="166.92516875" y1="106.25" x2="166.92516875" y2="104.25" width="0.001" layer="20"/>
+<wire x1="156.92516875" y1="106.25" x2="166.92516875" y2="106.25" width="0.001" layer="20"/>
+<wire x1="290.06295" y1="106.25" x2="290.06295" y2="104.25" width="0.001" layer="20"/>
+<wire x1="300.06295" y1="106.25" x2="300.06295" y2="104.25" width="0.001" layer="20"/>
+<wire x1="290.06295" y1="106.25" x2="300.06295" y2="106.25" width="0.001" layer="20"/>
+<wire x1="23.57501875" y1="104.25" x2="10.05" y2="104.25" width="0.001" layer="20"/>
+<wire x1="33.57501875" y1="104.25" x2="156.92516875" y2="104.25" width="0.001" layer="20"/>
+<wire x1="166.92516875" y1="104.25" x2="290.06295" y2="104.25" width="0.001" layer="20"/>
+<wire x1="300.06295" y1="104.25" x2="313.80035" y2="104.25" width="0.001" layer="20"/>
 </plain>
 <attributes>
@@
 <wire x1="281.2024" y1="59.69" x2="278.60625" y2="54.0225" width="0" layer="19" extent="1-16"/>
 </signal>
-<signal name="N$42">
-<contactref element="MACRO_2" pad="MX1"/>
-<contactref element="D42" pad="A"/>
-<wire x1="312.16" y1="59.69" x2="309.5625" y2="54.0225" width="0" layer="19" extent="1-16"/>
-</signal>
 <signal name="N$43">
 <contactref element="L_SHIFT" pad="MX1"/>
@@
 <contactref element="D26" pad="C"/>
 <contactref element="D27" pad="C"/>
+<contactref element="D69" pad="C"/>
 <wire x1="147.6375" y1="69.8025" x2="166.6875" y2="69.8025" width="0" layer="19" extent="16-16"/>
 <wire x1="128.5875" y1="69.8025" x2="147.6375" y2="69.8025" width="0" layer="19" extent="16-16"/>
@@
 <wire x1="261.9375" y1="69.8025" x2="242.8875" y2="69.8025" width="0" layer="19" extent="16-16"/>
 <wire x1="285.75" y1="69.8025" x2="261.9375" y2="69.8025" width="0" layer="19" extent="16-16"/>
+<wire x1="309.5625" y1="69.8025" x2="285.75" y2="69.8025" width="0" layer="19" extent="16-16"/>
 <wire x1="28.575" y1="69.8025" x2="52.3875" y2="69.8025" width="0" layer="19" extent="16-16"/>
 </signal>
 <signal name="ROW2">
 <contactref element="D29" pad="C"/>
-<contactref element="D42" pad="C"/>
 <contactref element="D30" pad="C"/>
 <contactref element="D31" pad="C"/>
@@
 <contactref element="D40" pad="C"/>
 <contactref element="D41" pad="C"/>
+<contactref element="D42" pad="C"/>
 <wire x1="171.45" y1="50.7525" x2="190.5" y2="50.7525" width="0" layer="19" extent="16-16"/>
 <wire x1="152.4" y1="50.7525" x2="171.45" y2="50.7525" width="0" layer="19" extent="16-16"/>
@@
 <signal name="ROW4">
 <contactref element="D57" pad="C"/>
-<contactref element="D69" pad="C"/>
 <contactref element="D58" pad="C"/>
 <contactref element="D59" pad="C"/>
 <contactref element="D60" pad="C"/>
 <contactref element="D61" pad="C"/>
-<contactref element="D68" pad="C"/>
 <contactref element="D62" pad="C"/>
 <contactref element="D63" pad="C"/>
@@
 <wire x1="50.00625" y1="12.6525" x2="73.81875" y2="12.6525" width="0" layer="19" extent="16-16"/>
 <wire x1="26.19375" y1="12.6525" x2="50.00625" y2="12.6525" width="0" layer="19" extent="16-16"/>
-<wire x1="309.5625" y1="69.8025" x2="309.5625" y2="12.6525" width="0" layer="19" extent="16-16"/>
-<wire x1="309.5625" y1="88.8525" x2="309.5625" y2="69.8025" width="0" layer="19" extent="16-16"/>
 </signal>
 <signal name="ROW0">
@@
 <contactref element="D12" pad="C"/>
 <contactref element="D13" pad="C"/>
+<contactref element="D68" pad="C"/>
 <wire x1="138.1125" y1="88.8525" x2="157.1625" y2="88.8525" width="0" layer="19" extent="16-16"/>
 <wire x1="119.0625" y1="88.8525" x2="138.1125" y2="88.8525" width="0" layer="19" extent="16-16"/>
@@
 <wire x1="252.4125" y1="88.8525" x2="233.3625" y2="88.8525" width="0" layer="19" extent="16-16"/>
 <wire x1="280.9875" y1="88.8525" x2="252.4125" y2="88.8525" width="0" layer="19" extent="16-16"/>
+<wire x1="309.5625" y1="88.8525" x2="280.9875" y2="88.8525" width="0" layer="19" extent="16-16"/>
 </signal>
 <signal name="N$70">
@@
 </signal>
 <signal name="N$76">
-<contactref element="MACRO_0" pad="MX2"/>
 <contactref element="N" pad="MX2"/>
 <contactref element="SIX" pad="MX2"/>
@@
 <wire x1="141.5476" y1="62.23" x2="136.785" y2="81.28" width="0" layer="19" extent="1-1"/>
 <wire x1="151.0726" y1="43.18" x2="141.5476" y2="62.23" width="0" layer="19" extent="1-1"/>
-<wire x1="298.71" y1="100.33" x2="151.0726" y2="43.18" width="0" layer="19" extent="1-1"/>
 </signal>
 <signal name="N$77">
@@
 </signal>
 <signal name="N$78">
-<contactref element="MACRO_1" pad="MX2"/>
 <contactref element="COMMA" pad="MX2"/>
 <contactref element="EIGHT" pad="MX2"/>
@@
 <wire x1="189.1726" y1="43.18" x2="179.6476" y2="62.23" width="0" layer="19" extent="1-1"/>
 <wire x1="165.36" y1="100.33" x2="174.885" y2="81.28" width="0" layer="19" extent="1-1"/>
-<wire x1="298.71" y1="81.28" x2="189.1726" y2="43.18" width="0" layer="19" extent="1-1"/>
 </signal>
 <signal name="N$79">
@@
 <wire x1="279.66" y1="24.13" x2="279.66" y2="43.18" width="0" layer="19" extent="1-1"/>
 </signal>
+<signal name="N$42">
+<contactref element="MACRO_2" pad="MX1"/>
+<contactref element="D42" pad="A"/>
+<wire x1="309.5625" y1="54.0225" x2="312.16" y2="59.69" width="0" layer="19" extent="1-16"/>
+</signal>
 <signal name="N$83">
 <contactref element="BACKSPACE" pad="MX2"/>
 <contactref element="RIGHT_ARROW" pad="MX2"/>
 <contactref element="BACKSLASH" pad="MX2"/>
-<contactref element="MACRO_2" pad="MX2"/>
 <contactref element="MACRO_3" pad="MX2"/>
 <wire x1="274.8974" y1="81.28" x2="270.1354" y2="100.33" width="0" layer="19" extent="1-1"/>
-<wire x1="298.71" y1="62.23" x2="274.8974" y2="81.28" width="0" layer="19" extent="1-1"/>
-<wire x1="298.71" y1="43.18" x2="298.71" y2="62.23" width="0" layer="19" extent="1-1"/>
+<wire x1="298.71" y1="43.18" x2="274.8974" y2="81.28" width="0" layer="19" extent="1-1"/>
 <wire x1="298.71" y1="24.13" x2="298.71" y2="43.18" width="0" layer="19" extent="1-1"/>
 </signal>
+<signal name="N$84">
+<contactref element="MACRO_0" pad="MX2"/>
+<contactref element="MACRO_2" pad="MX2"/>
+<contactref element="MACRO_1" pad="MX2"/>
+<wire x1="298.71" y1="81.28" x2="298.71" y2="100.33" width="0" layer="19" extent="1-1"/>
+<wire x1="298.71" y1="62.23" x2="298.71" y2="81.28" width="0" layer="19" extent="1-1"/>
+</signal>
 </signals>

Commit message: added MCU scheme + readme
Parts:
- added C1, C2, C3, C4: 0.1uF, Components:C0603
- added C5: 10uF, Components:C0603
- added C6: 1uF, Components:C0603
- added C7, C8: 22pF, Components:C0603
- added R1, R2: 22, Components:R0603
- added R3, R4: 10k, Components:R0603
- added SW1: SWITCH-SMD-EVP-BB2A9B00, Controller:SWITCH-SMD-EVP-BB2A9B00
- added U$1: ATMEGA32U4-QFN44, MCU:QFN-44
- added Y1: 16MHz, SparkFun-Clocks:CRYSTAL-SMD-2X2.5MM
- moved D14 9.53 mm to (271.5, 90.5)
- moved D54 9.53 mm to (254.8, 33.3)
- moved D11 9.53 mm to (204.8, 90.5)
- moved D12 9.53 mm to (223.8, 90.5)
- moved D13 9.53 mm to (242.9, 90.5)
- moved D16 9.53 mm to (42.9, 71.4)
- moved D20 9.53 mm to (119.1, 71.4)
- moved D22 9.53 mm to (157.2, 71.4)
- moved D23 9.53 mm to (176.2, 71.4)
- moved D24 9.53 mm to (195.3, 71.4)
- moved D25 9.53 mm to (214.3, 71.4)
- moved D27 9.53 mm to (252.4, 71.4)
- moved D31 9.53 mm to (66.7, 52.4)
- moved D32 9.53 mm to (85.7, 52.4)
- moved D35 9.53 mm to (142.9, 52.4)
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Connections:
- new net D+: R2.1
- new net D-: R1.1
- new net GND: C1.1, C2.1, C3.1, C4.1, C5.1, C6.1, C7.1, C8.1, R4.1, SW1.A@1, SW1.A@2, U$1.15, U$1.23, U$1.35, U$1.43, U$1.5, U$1.TAB, Y1.P2, Y1.P4
- new net N$85: R4.2, U$1.33
- new net N$86: R3.2, SW1.B@3, SW1.B@4, U$1.13
- new net N$87: C7.2, U$1.17, Y1.P1
- new net N$88: C8.2, U$1.16, Y1.P3
- new net N$89: R2.2, U$1.4
- new net N$90: R1.2, U$1.3
- new net N$91: C6.2, U$1.6
- new net VCC: C1.2, C2.2, C3.2, C4.2, C5.2, R3.1, U$1.14, U$1.2, U$1.24, U$1.34, U$1.44, U$1.7
- net N$73: now also L_SPACE.MX2
- net N$74: no longer L_SPACE.MX2
Routing:
- net ROW4: track 0.00 -> 288.4 mm
- net ROW0: track 0.00 -> 287.0 mm
- net ROW1: track 0.00 -> 281.0 mm
- net ROW2: track 0.00 -> 279.8 mm
- net ROW3: track 0.00 -> 274.8 mm
- net N$71: track 0.00 -> 106.5 mm, vias 0 -> 8
- net N$82: track 0.00 -> 105.0 mm, vias 0 -> 8
- net N$72: track 0.00 -> 101.2 mm, vias 0 -> 8
- net N$80: track 0.00 -> 100.2 mm, vias 0 -> 8
- net N$81: track 0.00 -> 97.7 mm, vias 0 -> 8
- net N$83: track 0.00 -> 96.7 mm, vias 0 -> 4
- net N$79: track 0.00 -> 93.1 mm, vias 0 -> 8
- net N$77: track 0.00 -> 93.1 mm, vias 0 -> 8
- net N$75: track 0.00 -> 93.1 mm, vias 0 -> 8
- net N$73: track 0.00 -> 93.1 mm, vias 0 -> 8
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
Commit message: added USB-C + ferrite beads
Parts:
- added FB1, FB2, FB3, FB4, FB5, FB6: 50@100 MHz, Filter:BEADC1608X95N
- added J1, J2, J3: TYPE-C-31-M-12, TYPE-C-31-M-12:HRO_TYPE-C-31-M-12
- added R10, R5, R6, R7, R8, R9: 5.1k, Components:R0603
- moved C6 198.1 mm to (176.5, -93.5), flipped to the bottom
- moved R2 187.0 mm to (165.3, 25.0), flipped to the bottom
- moved R1 183.1 mm to (162.3, 25.0), flipped to the bottom
- moved U$1 165.6 mm to (160.5, 19.5), flipped to the bottom, turned to 315 degrees
- moved C1 164.1 mm to (156.5, -7.00), flipped to the bottom
- moved C2 163.7 mm to (155.5, -21.5), flipped to the bottom
- moved C3 158.3 mm to (149.0, -33.0), flipped to the bottom
- moved C4 156.9 mm to (144.5, -52.0), flipped to the bottom
- moved C5 153.9 mm to (138.0, -66.5), flipped to the bottom
- moved C7 146.4 mm to (112.0, -108.0), flipped to the bottom
- moved C8 124.7 mm to (86.0, -109.5), flipped to the bottom
- moved Y1 121.4 mm to (109.0, -44.0), flipped to the bottom
- moved R3 120.0 mm to (107.5, -60.0), flipped to the bottom
- moved SW1 60.4 mm to (49.7, -16.9), flipped to the bottom
- moved R4 50.4 mm to (28.0, -76.5), flipped to the bottom
Connections:
- new net +5V: FB1.2, FB2.2, FB4.2
- new net N$100: FB6.1, J3.S1, J3.S2, J3.S3, J3.S4
- new net N$92: J2.A5, R7.1
- new net N$93: J1.A5, R5.1
- new net N$94: J1.B5, R6.1
- new net N$95: J2.B5, R8.1
- new net N$96: FB5.1, J2.S1, J2.S2, J2.S3, J2.S4
- new net N$97: J3.A5, R9.1
- new net N$98: FB3.1, J1.S1, J1.S2, J1.S3, J1.S4
- new net N$99: J3.B5, R10.1
- new net VBUS: FB1.1, FB2.1, FB4.1, J1.A4B9, J1.B4A9, J2.A4B9, J2.B4A9, J3.A4B9, J3.B4A9
- net D+: now also J1.A6, J1.B6, J2.A6, J2.B6, J3.A6, J3.B6
- net D-: now also J1.A7, J1.B7, J2.A7, J2.B7, J3.A7, J3.B7
- net GND: now also FB3.2, FB5.2, FB6.2, J1.A1B12, J1.B1A12, J2.A1B12, J2.B1A12, J3.A1B12, J3.B1A12, R10.2, R5.2, R6.2, R7.2, R8.2, R9.2
Other:
- board size 307.8 x 96.2 mm -> 307.8 x 101.2 mm
